File: FlexiblePS/FlexiblePS.kicad_pcb (KiCad board)
At the start: 2 copper layers, 99.3 x 98.6 mm, 118 parts, among them J1 Conn_01x02, J10 Conn_01x01, J11 Conn_01x01, J12 Conn_01x04, J13 Conn_01x02, J14 Conn_01x02, J15 Conn_01x02, J2 Conn_02x03_Odd_Even, J3 Conn_01x02, J4 Conn_01x02, J5 Conn_01x02, J6 Conn_01x01, J7 Conn_01x01, J8 Conn_01x02, J9 Conn_01x02, Q1 TIP42, Q2 TIP41, Q3 2N3906, Q4 TIP41C, U1 ATMEGA328P-PU, U2 LM358, U3 LCD-016N002L, U4 TL494, U5 LMT85, U6 LMT85, U9 LM7805_TO220, X3 16MHz

Commit message: Renamed project to FlexiblePS
Parts:
- F1: footprint LiFePO4smartcharger:SL506Pfuseholder -> FlexiblePS:SL506Pfuseholder
- Q2: footprint LiFePO4smartcharger:TO-247_TO-3P_Vertical -> FlexiblePS:TO-247_TO-3P_Vertical
Changed lines of the file:
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@@
   )
   (setup
-    (last_trace_width 0.35)
+    (last_trace_width 0.204)
     (user_trace_width 0.35)
     (user_trace_width 0.5)
@@
     )
   )
-  (module LiFePO4smartcharger:TO-247_TO-3P_Vertical (layer F.Cu)
+  (module FlexiblePS:TO-247_TO-3P_Vertical (layer F.Cu)
     (at 51.78 51.28 90)
     (descr "TO-247, Vertical, RM 5.45mm, TO-3P, TO-220")
@@
     )
   )
-  (module LiFePO4smartcharger:SL506Pfuseholder (layer F.Cu)
+  (module FlexiblePS:SL506Pfuseholder (layer F.Cu)
     (at 61.96 116.6)
     (fp_text reference F1 (at 0 0 90) (layer F.SilkS)
